Commit message: se actualiza modelo jaime

File: src/kobuki/kobuki_description/urdf/kobuki.urdf.xacro (robot description, xacro)
@@ -213,10 +213,10 @@
     </link>
     <!-- kobuki agrega link_palo y base-->
-    <joint name="camara_joint" type="fixed">
+    <!--joint name="camara_joint" type="fixed">
       <axis xyz="0 1 0" />
       <origin xyz="0 0 0.8" rpy="0 0 0"/>
       <parent link="link_palo"/>
       <child link="camara"/>
-    </joint>
+    </joint-->
     <!--joint camara de profunidad-->
     <joint name="camara_profundidad_joint" type="fixed">
@@ -228,30 +228,28 @@
     </joint>
     <joint name="camara_profundidad_optical_joint" type="fixed">
-  <origin xyz="0 0 0" rpy="${-M_PI/2} 0 ${-M_PI/2}" />
-  <parent link="camara_profundidad" />
-  <child link="camara_profundidad_optical" />
-</joint>
-<link name="camara_profundidad_optical"/>
-    <link name="camara">
-      <!--collision>
-        <origin xyz="0 0 0" rpy="0 0 0"/>
-        <geometry>
-      <box size="${camara ${camara} ${camara}"/>
-        </geometry>
-      </collision-->
-      <visual>
-        <origin xyz="0 0 0" rpy="0 0 0"/>
-        <geometry>
+      <origin xyz="0 0 0" rpy="${-M_PI/2} 0 ${-M_PI/2}" />
+      <parent link="camara_profundidad" />
+      <child link="camara_profundidad_optical" />
+    </joint>
+<!--link name="camara_profundidad_optical"/-->
+    <link name="camara_profundidad_optical">
+      <visual>
+        <origin xyz="0 0 0" rpy="0 0 0"/>
+        <geometry>
+          <!--mesh filename="package://kobuki_description/meshes/camera_ASUS_XTION.STL"/-->
           <!--box size="${camara} ${camara} ${camara}"/-->
-          <mesh filename="package://kobuki_description/meshes/camera_ASUS_XTION.STL"/>
+          <box size="0 0 0"/>
         </geometry>
         <material name="red"/>
       </visual>
-      <!--inertial>
-        <mass value="1e-5" />
-        <origin xyz="0 0 0" rpy="0 0 0"/>
-        <inertia ixx="1e-6" ixy="0" ixz="0" iyy="1e-6" iyz="0" izz="1e-6" />
-      </inertial-->
-    </link>
+    </link>
+    <!--link name="camara_profundidad_optical"/>
+      <visual>
+        <origin xyz="0 0 0" rpy="0 0 0"/>
+        <geometry>
+          <box size="${camara} ${camara} ${camara}"/>
+        </geometry>
+      </visual>
+    </link-->
     <!--camara de profunidad, kinetic microsoft-->
     <link name="camara_profundidad" type="fixed">

Commit message: se agrega structure

File: src/kobuki/kobuki_description/urdf/kobuki.urdf.xacro (robot description, xacro)
@@ -319,4 +319,17 @@
       <child link="wood_base"/>
     </joint>
+    <!--link name="structure" type="fixed">
+      <visual>
+        <geometry>
+          <mesh filename="package://kobuki_description/meshes/structure_link.STL"/>
+        </geometry>
+        <origin xyz="0 0 0" rpy="0 0 0"/>
+      </visual>
+    </link-->
+    <!--joint name="structure_to_base" type="fixed">
+      <origin xyz="0 0 0"/>
+      <parent link="base_link"/>
+      <child link="structure"/>
+    </joint-->
     <!-- Kobuki Gazebo simulation details -->
     <kobuki_sim/>

Commit message: se actualiza modelo y se prueba scane

File: src/kobuki/kobuki_description/urdf/kobuki.urdf.xacro (robot description, xacro)
@@ -11,5 +11,5 @@
   <xacro:include filename="$(find kobuki_description)/urdf/common_properties.urdf.xacro"/>
   <xacro:include filename="$(find kobuki_description)/urdf/kobuki_gazebo.urdf.xacro"/>
-  <xacro:property name="camara" value="0.05" />
+  <xacro:property name="camara" value="0.0001" />
   <xacro:property name="M_PI" value="3.1415926535897931" />
   <!-- Kobuki -->
@@ -222,7 +222,8 @@
     <joint name="camara_profundidad_joint" type="fixed">
       <!--axis xyz="0 1 0" /-->
-      <origin xyz ="0.1 0 0.15" rpy="0 0 0"/>  <!--heght480-640/2-->
+      <origin xyz="0.12 0 0.352" rpy="0 -0.00031618 0" />  <!--heght480-640/2-->
       <!--parent link="base_link"/-->
-      <parent link="pc_base_up"/>
+      <!--parent link="pc_base_up"/-->
+      <parent link="structure"/>
       <child link="camara_profundidad"/>
     </joint>
@@ -238,6 +239,6 @@
         <geometry>
           <!--mesh filename="package://kobuki_description/meshes/camera_ASUS_XTION.STL"/-->
-          <!--box size="${camara} ${camara} ${camara}"/-->
-          <box size="0 0 0"/>
+          <box size="${camara} ${camara} ${camara}"/>
+          <!--box size="0 0 0"/-->
         </geometry>
         <material name="red"/>
@@ -263,47 +264,4 @@
       </visual>
     </link>
-    <link name="link_palo" type="fixed">
-      <visual>
-        <geometry>
-          <cylinder length="1.42" radius="0.0125"/>
-          <material name="black">
-            <color rgba="0.1 0.1 0.1 1"/>
-          </material>
-        </geometry>
-        <origin xyz="0 0 0" rpy="0 0 0"/>
-      </visual>
-    </link>
-    <!--joint name="link_palo_base" type="fixed"-->
-    <joint name="link_palo_to_pc_base_up" type="fixed">
-      <origin xyz="0 0 0.8"/>
-      <parent link="pc_base_up"/>
-      <child link="link_palo"/>
-    </joint>
-    <link name="pc_base_down" type="fixed">
-      <visual>
-        <geometry>
-          <mesh filename="package://kobuki_description/meshes/pc_base_down.STL"/>
-        </geometry>
-        <origin xyz="0 0 0" rpy="0 0 0"/>
-      </visual>
-    </link>
-    <joint name="pc_base_down_to_base_link" type="fixed">
-      <origin xyz="0 0 0.1"/>
-      <parent link="base_link"/>
-      <child link="pc_base_down"/>
-    </joint>
-    <link name="pc_base_up" type="fixed">
-      <visual>
-        <geometry>
-          <mesh filename="package://kobuki_description/meshes/pc_base_up.STL"/>
-        </geometry>
-        <origin xyz="0 0 0" rpy="0 0 0"/>
-      </visual>
-    </link>
-    <joint name="pc_base_up_to_base_link" type="fixed">
-      <origin xyz="0 0 0.18"/>
-      <parent link="base_link"/>
-      <child link="pc_base_up"/>
-    </joint>
     <link name="wood_base" type="fixed">
       <visual>
@@ -319,17 +277,18 @@
       <child link="wood_base"/>
     </joint>
-    <!--link name="structure" type="fixed">
+    <link name="structure" type="fixed">
       <visual>
         <geometry>
           <mesh filename="package://kobuki_description/meshes/structure_link.STL"/>
         </geometry>
-        <origin xyz="0 0 0" rpy="0 0 0"/>
-      </visual>
-    </link-->
-    <!--joint name="structure_to_base" type="fixed">
-      <origin xyz="0 0 0"/>
+        <origin xyz="0.00168628472042168 -2.03976137341799E-07 0.150942765196013" rpy="0 0 0"/>
+      </visual>
+    </link>
+    <joint name="structure_to_base" type="fixed">
+      <origin xyz="0 0 -0.07"/>
       <parent link="base_link"/>
       <child link="structure"/>
-    </joint-->
+      <axis xyz="0 0 1" />
+    </joint>
     <!-- Kobuki Gazebo simulation details -->
     <kobuki_sim/>

Commit message: se agrega hokuyo

File: src/kobuki/kobuki_description/urdf/kobuki.urdf.xacro (robot description, xacro)
@@ -219,8 +219,8 @@
       <child link="camara"/>
     </joint-->
-    <!--joint camara de profunidad-->
+    <!--joint camara de profunidad-0.00031618-->
     <joint name="camara_profundidad_joint" type="fixed">
       <!--axis xyz="0 1 0" /-->
-      <origin xyz="0.12 0 0.352" rpy="0 -0.00031618 0" />  <!--heght480-640/2-->
+      <origin xyz="0.12 0 0.352" rpy="0 ${M_PI/11} 0" />  <!--heght480-640/2-->
       <!--parent link="base_link"/-->
       <!--parent link="pc_base_up"/-->
@@ -264,4 +264,18 @@
       </visual>
     </link>
+    <!--agrega laser hokuyo-->
+    <link name="hokuyo_link" type="fixed">
+      <visual>
+        <origin xyz="0 0 0" rpy="${M_PI/2} 0 ${M_PI/2}"/>
+        <geometry>
+          <mesh filename="package://kobuki_description/meshes/Hokuyo_UST_10LX.STL"/>
+        </geometry>
+      </visual>
+    </link>
+    <joint name="hokuyo_to_wood_base_link" type="fixed">
+      <origin xyz="0.11 0 0.11"/>
+      <parent link="wood_base"/>
+      <child link="hokuyo_link"/>
+    </joint>
     <link name="wood_base" type="fixed">
       <visual>
